File: VolumeControl/VolumeControl.kicad_sch (KiCad schematic)
At the start: 63 parts, among them J1 Barrel_Jack, J12 Conn_01x03, J13 Conn_01x03, J2 Conn_01x03, J3 Conn_01x03, J4 Conn_01x03, J8 Conn_01x03, J9 Conn_01x03, U1 OPA1612AxD, U10 LM1117MP-5.0, U2 MCP4251-xxxx-SL, U3 L7812, U4 MCP4251-xxxx-SL, U5 OPA1612AxD, U6 MCP4251-xxxx-SL, U7 OPA1612AxD, U8 OPA1612AxD, U9 WEMOS_D1_mini

Commit message: PPT first draft
Parts:
- removed A1: RaspberryPi_Pico_W, Module:RaspberryPi_Pico_W_SMD, symbol MCU_Module:RaspberryPi_Pico_W_Extensive
- removed U9: WEMOS_D1_mini, RF_Module:WEMOS_D1_mini_light, symbol RF_Module:WEMOS_D1_mini
- added D3, D4, D5, D6, D7, D8: LED, LED_SMD:LED_1210_3225Metric, symbol Device:LED
- added J5: XLR3_Ground, symbol Connector_Audio:XLR3_Ground
- added R10, R18, R4, R5, R6, R9: 100R, Resistor_SMD:R_0805_2012Metric, symbol Device:R
- added R19, R20, R21: 10K, Resistor_SMD:R_0805_2012Metric, symbol Device:R
- added SW1: Select, Button_Switch_SMD:SW_SPST_PTS647_Sx50, symbol Switch:SW_Push
- added SW2: Up, Button_Switch_SMD:SW_SPST_PTS647_Sx50, symbol Switch:SW_Push
- added SW3: Down, Button_Switch_SMD:SW_SPST_PTS647_Sx50, symbol Switch:SW_Push
- added U12: ESP32-S3-DevKitC, Espressif:ESP32-S3-DevKitC, symbol Espressif:ESP32-S3-DevKitC
Connections:
- net GND: now also R10.2, R18.2, R4.2, R5.2, R6.2, R9.2, SW1.2, SW2.2, SW3.2, U12.22 (GND), U12.23 (GND), U12.24 (GND), U12.44 (GND)
- net SCK: now also U2.2 (SCK), U4.2 (SCK), U6.2 (SCK), U12.18 (GPIO12/ADC2_CH1)
- net V5V: now also U12.21 (5V)
- net CS1: now reaches U4.1 (~{CS})
- net MISO: now reaches U4.13 (SDO)
- net MISO: now also U2.13 (SDO), U6.13 (SDO), U12.19 (GPIO13/ADC2_CH2)
- net MOSI: now reaches U4.3 (SDI)
- net MOSI: now also U2.3 (SDI), U6.3 (SDI), U12.17 (GPIO11/ADC2_CH0)
- net CS2: now reaches U6.1 (~{CS})
- net CS0: now reaches U2.1 (~{CS})
- net CS0: now also U12.16 (GPIO10/ADC1_CH9)
- new net: C10.2, U4.7 (P1A)
- new net: D6.1 (K), R9.1
- new net: D5.1 (K), R6.1
- new net: D7.1 (K), R10.1
- new net: D8.1 (K), R18.1
- new net: D4.1 (K), R5.1
- new net: C8.2, U2.7 (P1A)
- new net: D3.1 (K), R4.1
- new net Down: R21.2, SW3.1
- new net LED1: D3.2 (A)
- new net LED2: D4.2 (A)
- new net LED3: D5.2 (A)
- new net LED4: D6.2 (A)
- new net LED5: D7.2 (A)
- new net LED6: D8.2 (A)
- new net Select: R19.2, SW1.1
- new net UP: R20.2, SW2.1
- new net V3V: R19.1, R20.1, R21.1, U12.1 (3V3), U12.2 (3V3)
Other:
- moved on the sheet: C10, C11, C16, C17, C8, C9, J2, R3
